File: relayBoard/relayChannel.sch (KiCad schematic (older format))
At the start: 5 parts, among them K11 G6S-2, Q1 Q_NMOS_DGS

Commit message: first pass at revisions
Parts:
- added C?: C, symbol Device:C
- added D?: D_Zener, symbol Device:D_Zener
- K11: footprint Relay_SMD:Relay_DPDT_Omron_G6SK-2G -> Relay_THT:Relay_DPDT_Omron_G6S-2
Connections:
- net GND: now also C?.2, D?.2 (A)
- net at Q1.1 (G), R4.1: now also D?.1 (K)
- net at K11.1, R5.1: now also C?.1
Other:
- moved on the sheet: D11, Q?, R?
