File: relayBoard/relayBoard.sch (KiCad schematic (older format))
At the start: 33 parts, among them J1 Conn_01x10, J10 Conn_02x07_Odd_Even, J11 Conn_01x10, J12 Conn_01x10, J13 Conn_01x10, J14 DB50_CON, J2 Conn_01x10, J3 Conn_01x01, J4 Conn_01x01, J5 Conn_01x01, J6 Conn_01x01, J7 Conn_01x01, J8 Conn_01x01, J9 Conn_02x07_Odd_Even, U1 PI4IOE5V96248

Commit message: first pass at revisions
Parts:
- removed C1, C2, C3: 1u, Resistor_SMD:R_0603_1608Metric_Pad1.05x0.95mm_HandSolder, symbol Device:C
- removed J1, J11, J12, J13, J2: Conn_01x10, Connector_JST:JST_EH_S10B-EH_1x10_P2.50mm_Horizontal, symbol Connector_Generic:Conn_01x10
- removed J10, J9: Conn_02x07_Odd_Even, Connector_PinHeader_2.00mm:PinHeader_2x07_P2.00mm_Vertical, symbol Connector_Generic:Conn_02x07_Odd_Even
- removed J14: DB50_CON, Connector_Dsub:DB50_CON, symbol cLib:DB50_CON
- removed JP1, JP2, JP3: Jumper_3_Bridged12, Connector_PinHeader_2.00mm:PinHeader_1x03_P2.00mm_Vertical, symbol Jumper:Jumper_3_Bridged12
- removed JP4: Jumper_2_Bridged, Connector_PinHeader_2.54mm:PinHeader_1x02_P2.54mm_Vertical, symbol Jumper:Jumper_2_Bridged
- removed R1, R2, R3: 10K, Resistor_SMD:R_0603_1608Metric_Pad1.05x0.95mm_HandSolder, symbol Device:R
- removed R84, R85: 10k, Resistor_SMD:R_0603_1608Metric_Pad1.05x0.95mm_HandSolder, symbol Device:R
- removed U1: PI4IOE5V96248, Package_DFN_QFN:QFN-56-1EP_7x7mm_P0.4mm_EP5.6x5.6mm, symbol cLib:PI4IOE5V96248
- added J? (x6): Conn_02x04_Top_Bottom, symbol Connector_Generic:Conn_02x04_Top_Bottom
Connections:
- net labels added: +5V, C20, H0, H1, H10, H11, H12, H13, H14, H15, H16, H17, H18, H19, H2, H20, H3, H4, H5, H6, H7, H8, H9, HV_SW, I0, I1, I10, I11, I12, I13, I14, I15, I16, I17, I18, I19, I2, I20, I3, I4, I5, I6, I7, I8, I9, IN0, IN1, IN10, IN11, IN12, IN13, IN14, IN15, IN16, IN17, IN18, IN19, IN2, IN20, IN3, IN4, IN5, IN6, IN7, IN8, IN9, INPUT_1, INPUT_2, OUT20
- net labels removed: 5V, 5V_LIN, A0, A1, A2, E0, E0B, E1, E10, E10B, E11, E11B, E12, E12B, E13, E13B, E14, E14B, E15, E15B, E16, E16B, E17, E17B, E18, E18B, E19, E19B, E1B, E2, E2B, E3, E3B, E4, E4B, E5, E5B, E6, E6B, E7, E7B, E8, E8B, E9, E9B, EX0, EX1, EX2, EX3, EX4, EX5, EX6, EX7, HV, INT_N, RST_N, SCL, SDA
- wire segments 499 -> 523
Other:
- moved on the sheet: H1, H2, H3, H4, H5, H6, J3, J4, J5, J6, J7, J8

Commit message: First pass layout finished
Parts:
- J10, J11, J12, J7, J8, J9: renamed from J?; footprint (none) -> Connector_Molex:Molex_Micro-Fit_3.0_43045-0800_2x04_P3.00mm_Horizontal
- renumbered J3 to J1, J4 to J2, J5 to J3, J6 to J4, J7 to J5, J8 to J6
Connections:
- net INPUT_2: no longer J5.1 (Pin_1)
- net OUT0: now also J10.4 (Pin_4), J10.8 (Pin_8); no longer J10.1 (Pin_1), J10.5 (Pin_5)
- net OUT1: now also J10.3 (Pin_3); no longer J10.2 (Pin_2)
- net OUT10: now also J11.2 (Pin_2); no longer J11.3 (Pin_3)
- net OUT11: now also J11.6 (Pin_6); no longer J11.7 (Pin_7)
- net OUT12: now also J11.1 (Pin_1); no longer J11.4 (Pin_4)
- net OUT13: now also J11.5 (Pin_5); no longer J11.8 (Pin_8)
- net OUT14: now also J12.4 (Pin_4), J12.8 (Pin_8); no longer J12.1 (Pin_1), J12.5 (Pin_5)
- net OUT15: now also J12.3 (Pin_3); no longer J12.2 (Pin_2)
- net OUT16: now also J12.7 (Pin_7); no longer J12.6 (Pin_6)
- net OUT17: now also J12.2 (Pin_2); no longer J12.3 (Pin_3)
- net OUT18: now also J12.6 (Pin_6); no longer J12.7 (Pin_7)
- net OUT19: now also J12.1 (Pin_1); no longer J12.4 (Pin_4)
- net OUT2: now also J10.7 (Pin_7); no longer J10.6 (Pin_6)
- net OUT20: now also J12.5 (Pin_5); no longer J12.8 (Pin_8)
- net OUT3: now also J10.2 (Pin_2); no longer J10.3 (Pin_3)
- net OUT4: now also J10.6 (Pin_6); no longer J10.7 (Pin_7)
- net OUT5: now also J10.1 (Pin_1); no longer J10.4 (Pin_4)
- net OUT6: now also J10.5 (Pin_5); no longer J10.8 (Pin_8)
- net OUT7: now also J11.4 (Pin_4), J11.8 (Pin_8); no longer J11.1 (Pin_1), J11.5 (Pin_5)
- net OUT8: now also J11.3 (Pin_3); no longer J11.2 (Pin_2)
- net OUT9: now also J11.7 (Pin_7); no longer J11.6 (Pin_6)
- new net INPUT_2_IN: J5.1 (Pin_1)

Commit message: updates to connector connections and converter transformer
Parts:
- added J19, J20: Conn_02x04_Top_Bottom, Connector_Molex:Molex_Micro-Fit_3.0_43045-0800_2x04_P3.00mm_Horizontal, symbol Connector_Generic:Conn_02x04_Top_Bottom
Connections:
- net IN10: now also J8.7 (Pin_7); no longer J8.3 (Pin_3)
- net IN11: now also J8.4 (Pin_4); no longer J8.7 (Pin_7)
- net IN12: now also J8.8 (Pin_8), J9.1 (Pin_1), J9.5 (Pin_5); no longer J8.4 (Pin_4)
- net IN13: now also J9.2 (Pin_2); no longer J8.8 (Pin_8)
- net IN14: now also J9.6 (Pin_6); no longer J9.1 (Pin_1), J9.5 (Pin_5)
- net IN15: now also J9.3 (Pin_3); no longer J9.2 (Pin_2)
- net IN16: now also J9.7 (Pin_7); no longer J9.6 (Pin_6)
- net IN17: now also J9.4 (Pin_4); no longer J9.3 (Pin_3)
- net IN18: now also J9.8 (Pin_8), J19.1 (Pin_1), J19.5 (Pin_5); no longer J9.7 (Pin_7)
- net IN19: now also J19.2 (Pin_2); no longer J9.4 (Pin_4)
- net IN20: now also J19.6 (Pin_6); no longer J9.8 (Pin_8)
- net IN6: now also J8.1 (Pin_1), J8.5 (Pin_5)
- net IN7: now also J8.2 (Pin_2); no longer J8.1 (Pin_1), J8.5 (Pin_5)
- net IN8: now also J8.6 (Pin_6); no longer J8.2 (Pin_2)
- net IN9: now also J8.3 (Pin_3); no longer J8.6 (Pin_6)
- net OUT10: now also J11.6 (Pin_6); no longer J11.2 (Pin_2)
- net OUT11: now also J11.1 (Pin_1); no longer J11.6 (Pin_6)
- net OUT12: now also J11.5 (Pin_5), J12.4 (Pin_4), J12.8 (Pin_8); no longer J11.1 (Pin_1)
- net OUT13: now also J12.3 (Pin_3); no longer J11.5 (Pin_5)
- net OUT14: now also J12.7 (Pin_7); no longer J12.4 (Pin_4), J12.8 (Pin_8)
- net OUT15: now also J12.2 (Pin_2); no longer J12.3 (Pin_3)
- net OUT16: now also J12.6 (Pin_6); no longer J12.7 (Pin_7)
- net OUT17: now also J12.1 (Pin_1); no longer J12.2 (Pin_2)
- net OUT18: now also J12.5 (Pin_5), J20.4 (Pin_4), J20.8 (Pin_8); no longer J12.6 (Pin_6)
- net OUT19: now also J20.3 (Pin_3); no longer J12.1 (Pin_1)
- net OUT20: now also J20.7 (Pin_7); no longer J12.5 (Pin_5)
- net OUT6: now also J11.4 (Pin_4), J11.8 (Pin_8)
- net OUT7: now also J11.3 (Pin_3); no longer J11.4 (Pin_4), J11.8 (Pin_8)
- net OUT8: now also J11.7 (Pin_7); no longer J11.3 (Pin_3)
- net OUT9: now also J11.2 (Pin_2); no longer J11.7 (Pin_7)
Changed lines of the file:
@@
 EESchema Schematic File Version 4
-LIBS:relayBoard-cache
-EELAYER 29 0
+EELAYER 30 0
 EELAYER END
 $Descr B 17000 11000
@@
 IN6
 Text Label 800  3100 0    50   ~ 0
+IN6
+Text Label 1700 3100 0    50   ~ 0
+IN6
+Text Label 800  3200 0    50   ~ 0
 IN7
-Text Label 1700 3100 0    50   ~ 0
-IN7
-Text Label 800  3200 0    50   ~ 0
+Text Label 1700 3200 0    50   ~ 0
 IN8
-Text Label 1700 3200 0    50   ~ 0
+Text Label 800  3300 0    50   ~ 0
 IN9
-Text Label 800  3300 0    50   ~ 0
+Text Label 1700 3300 0    50   ~ 0
 IN10
-Text Label 1700 3300 0    50   ~ 0
+Text Label 800  3400 0    50   ~ 0
 IN11
-Text Label 800  3400 0    50   ~ 0
+Text Label 1700 3400 0    50   ~ 0
 IN12
-Text Label 1700 3400 0    50   ~ 0
+Text Label 800  3750 0    50   ~ 0
+IN12
+Text Label 1700 3750 0    50   ~ 0
+IN12
+Text Label 800  3850 0    50   ~ 0
 IN13
-Text Label 800  3750 0    50   ~ 0
+Text Label 1700 3850 0    50   ~ 0
 IN14
-Text Label 1700 3750 0    50   ~ 0
-IN14
-Text Label 800  3850 0    50   ~ 0
+Text Label 800  3950 0    50   ~ 0
 IN15
-Text Label 1700 3850 0    50   ~ 0
+Text Label 1700 3950 0    50   ~ 0
 IN16
-Text Label 800  3950 0    50   ~ 0
+Text Label 800  4050 0    50   ~ 0
 IN17
-Text Label 1700 3950 0    50   ~ 0
+Text Label 1700 4050 0    50   ~ 0
 IN18
-Text Label 800  4050 0    50   ~ 0
-IN19
-Text Label 1700 4050 0    50   ~ 0
-IN20
 Text Label 15350 2450 0    50   ~ 0
 OUT5
@@
 OUT0
 Text Label 15350 3100 0    50   ~ 0
+OUT11
+Text Label 16250 3100 0    50   ~ 0
 OUT12
-Text Label 16250 3100 0    50   ~ 0
+Text Label 16250 3200 0    50   ~ 0
+OUT10
+Text Label 16250 3400 0    50   ~ 0
+OUT6
+Text Label 15350 3750 0    50   ~ 0
+OUT17
+Text Label 16250 3750 0    50   ~ 0
+OUT18
+Text Label 15350 3850 0    50   ~ 0
+OUT15
+Text Label 16250 3850 0    50   ~ 0
+OUT16
+Text Label 15350 3950 0    50   ~ 0
 OUT13
-Text Label 15350 3200 0    50   ~ 0
-OUT10
-Text Label 16250 3200 0    50   ~ 0
-OUT11
-Text Label 15350 3300 0    50   ~ 0
-OUT8
-Text Label 16250 3300 0    50   ~ 0
-OUT9
-Text Label 15350 3400 0    50   ~ 0
-OUT7
-Text Label 16250 3400 0    50   ~ 0
-OUT7
-Text Label 15350 3750 0    50   ~ 0
-OUT19
-Text Label 16250 3750 0    50   ~ 0
-OUT20
-Text Label 15350 3850 0    50   ~ 0
-OUT17
-Text Label 16250 3850 0    50   ~ 0
-OUT18
-Text Label 15350 3950 0    50   ~ 0
-OUT15
 Text Label 16250 3950 0    50   ~ 0
-OUT16
+OUT14
 Text Label 15350 4050 0    50   ~ 0
-OUT14
+OUT12
 Text Label 16250 4050 0    50   ~ 0
-OUT14
+OUT12
 Wire Wire Line
 	5800 9650 5300 9650
 Text Label 5300 9650 0    50   ~ 0
 INPUT_2
+$Comp
+L Connector_Generic:Conn_02x04_Top_Bottom J19
+U 1 1 5F8C51E4
+P 1200 4500
+F 0 "J19" H 1250 4817 50  0000 C CNN
+F 1 "Conn_02x04_Top_Bottom" H 1250 4726 50  0000 C CNN
+F 2 "Connector_Molex:Molex_Micro-Fit_3.0_43045-0800_2x04_P3.00mm_Horizontal" H 1200 4500 50  0001 C CNN
+F 3 "~" H 1200 4500 50  0001 C CNN
+	1    1200 4500
+	1    0    0    -1
+$EndComp
+Wire Wire Line
+	1000 4400 800  4400
+Wire Wire Line
+	1500 4400 1700 4400
+Wire Wire Line
+	1500 4500 1700 4500
+Wire Wire Line
+	800  4500 1000 4500
+Text Label 800  4400 0    50   ~ 0
+IN18
+Text Label 1700 4400 0    50   ~ 0
+IN18
+Text Label 800  4500 0    50   ~ 0
+IN19
+Text Label 1700 4500 0    50   ~ 0
+IN20
+$Comp
+L Connector_Generic:Conn_02x04_Top_Bottom J20
+U 1 1 5FBF1EBB
+P 15750 4500
+F 0 "J20" H 15800 4817 50  0000 C CNN
+F 1 "Conn_02x04_Top_Bottom" H 15800 4726 50  0000 C CNN
+F 2 "Connector_Molex:Molex_Micro-Fit_3.0_43045-0800_2x04_P3.00mm_Horizontal" H 15750 4500 50  0001 C CNN
+F 3 "~" H 15750 4500 50  0001 C CNN
+	1    15750 4500
+	1    0    0    -1
+$EndComp
+Wire Wire Line
+	15550 4600 15350 4600
+Wire Wire Line
+	15550 4700 15350 4700
+Wire Wire Line
+	16250 4600 16050 4600
+Wire Wire Line
+	16250 4700 16050 4700
+Text Label 15350 4700 0    50   ~ 0
+OUT18
+Text Label 15350 3200 0    50   ~ 0
+OUT9
+Text Label 15350 3300 0    50   ~ 0
+OUT7
+Text Label 16250 3300 0    50   ~ 0
+OUT8
+Text Label 15350 3400 0    50   ~ 0
+OUT6
+Text Label 16250 4700 0    50   ~ 0
+OUT18
+Text Label 16250 4600 0    50   ~ 0
+OUT20
+Text Label 15350 4600 0    50   ~ 0
+OUT19
 $EndSCHEMATC
